Commit message: update description urdf

File: src/bumperbot_description/urdf/bumperbot.urdf.xacro (robot description, xacro)
@@ -13,5 +13,5 @@
             <geometry>
                 <!--extracting the mesh from file-->
-                <mesh filename="package://bumperbot_description/meshes/base_link.STL" scale="10.0"/>
+                <mesh filename="package://bumperbot_description/meshes/base_link.STL" scale="1.0"/>
             </geometry>
         </visual>
@@ -46,5 +46,5 @@
         </visual>
     </link>
-    <joint name="wheel_leftt_joint" type="continuous">
+    <joint name="wheel_left_joint" type="continuous">
         <parent link ="base_link"/>
         <child link="wheel_left_link"/>
@@ -56,5 +56,5 @@
             <origin rpy="0 0 0" xyz = "0 0 0"/>
             <geometry>
-                <mesh filename="package://bumperbot_description/meshes/castor_front_link.STL" scale="1.0"/>
+                <mesh filename="package://bumperbot_description/meshes/caster_front_link.STL" scale="1.0"/>
             </geometry>
         </visual>
@@ -69,5 +69,5 @@
             <origin rpy="0 0 0" xyz = "0 0 0"/>
             <geometry>
-                <mesh filename="package://bumperbot_description/meshes/castor_rear_link.STL" scale="1.0"/>
+                <mesh filename="package://bumperbot_description/meshes/caster_rear_link.STL" scale="1.0"/>
             </geometry>
         </visual>
